File: lipo_cell_protection.kicad_sch (KiCad schematic)
At the start: 12 parts, among them J1 V_CELL, J2 GND_CELL, J3 V_CELL, J4 V_CELL, Q1 PMZ600UNEYL, Q2 PMZ600UNEYL, U1 BQ29700DSER

Commit message: round attempt
Parts:
- J1, J2, J3, J4: footprint Connector_PinHeader_1.00mm:PinHeader_1x01_P1.00mm_Vertical -> TestPoint:TestPoint_Pad_D1.0mm
Changed lines of the file:
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@@
       (effects (font (size 1.27 1.27)))
     )
-    (property "Footprint" "Connector_PinHeader_1.00mm:PinHeader_1x01_P1.00mm_Vertical" (at 58.42 58.42 0)
+    (property "Footprint" "TestPoint:TestPoint_Pad_D1.0mm" (at 58.42 58.42 0)
       (effects (font (size 1.27 1.27)) hide)
     )
@@
       (effects (font (size 1.27 1.27)))
     )
-    (property "Footprint" "Connector_PinHeader_1.00mm:PinHeader_1x01_P1.00mm_Vertical" (at 58.42 60.96 0)
+    (property "Footprint" "TestPoint:TestPoint_Pad_D1.0mm" (at 58.42 60.96 0)
       (effects (font (size 1.27 1.27)) hide)
     )
@@
       (effects (font (size 1.27 1.27)))
     )
-    (property "Footprint" "Connector_PinHeader_1.00mm:PinHeader_1x01_P1.00mm_Vertical" (at 165.1 62.23 0)
+    (property "Footprint" "TestPoint:TestPoint_Pad_D1.0mm" (at 165.1 62.23 0)
       (effects (font (size 1.27 1.27)) hide)
     )
@@
       (effects (font (size 1.27 1.27)))
     )
-    (property "Footprint" "Connector_PinHeader_1.00mm:PinHeader_1x01_P1.00mm_Vertical" (at 165.1 59.69 0)
-      (effects (font (size 1.27 1.27)) hide)
-    )
+    (property "Footprint" "TestPoint:TestPoint_Pad_D1.0mm" (at 165.1 59.69 0)
+      (effects (font (size 1.27 1.27)) hide)
+    )

Commit message: full
Parts:
- removed R2, R3: 5M, Resistor_SMD:R_0201_0603Metric, symbol Device:R
- added J10, J8: SIG_2, TestPoint:TestPoint_Pad_D1.0mm, symbol Connector:Conn_01x01_Pin
- added J5: VCC, TestPoint:TestPoint_Pad_D1.0mm, symbol Connector:Conn_01x01_Pin
- added J6: GND, TestPoint:TestPoint_Pad_D1.0mm, symbol Connector:Conn_01x01_Pin
- added J7, J9: SIG_1, TestPoint:TestPoint_Pad_D1.0mm, symbol Connector:Conn_01x01_Pin
- J3: value V_CELL -> VCC
- J4: value V_CELL -> GND
Connections:
- net +BATT: now also J5.1 (Pin_1)
- net GND: now also J6.1 (Pin_1)
- new net SIG_1: J7.1 (Pin_1), J9.1 (Pin_1)
- new net SIG_2: J10.1 (Pin_1), J8.1 (Pin_1)
